Commit message: creating core urdf

File: description/robot_core.xacro (robot description, xacro)
@@ -1,4 +1,5 @@
 <?xml version="1.0"?>
 <robot xmlns:xacro="http://www.ros.org/wiki/xacro">
+    <xacro:include filename="inertial_macros.xacro"/>
             <!-- Farben -->
     <material name="white">
@@ -24,5 +25,5 @@
         <parent link="base_link"/>
         <child link="chassis"/>
-        <origin xyz="-0.1 0.0 0.0"/>
+        <origin xyz="-0.15 0.0 0.0"/>
     </joint>
     <link name="chassis">
@@ -32,13 +33,22 @@
                 <box size="0.3 0.3 0.15"/>
             </geometry>
-            <material name="black"/>
+            <material name="orange"/>
         </visual>
+        <collision>
+            <origin xyz="0.15 0.0 0.075"/>
+            <geometry>
+                <box size="0.3 0.3 0.15"/>
+            </geometry>
+        </collision>
+        <xacro:inertial_box mass="0.5" x="0.3" y="0.3" z="0.15">
+            <origion xyz="0.15 0.0 0.075" rpy="0.0 0.0 0.0"/>
+        </xacro:inertial_box>
     </link>
         <!-- LEFT WHEEL LINK -->
     <joint name="left_wheel_joint" type="continuous">
-        <origin xyz="0.0 0.0 0.0" rpy="0.0 0.0 0.0"/>
-        <parent link="parent_link"/>
-        <child link="child_link"/>
-        <axis xyz="0.0 0.0 0.0"/>
+        <origin xyz="0.0 0.175 0.0" rpy="-${pi/2} 0.0 0.0"/>
+        <parent link="base_link"/>
+        <child link="left_wheel"/>
+        <axis xyz="0.0 0.0 1.0"/>
         <limit lower="0.0" upper="0.0" effort="0.0" velocity="0.0"/>
     </joint>
@@ -46,10 +56,85 @@
         <visual>
             <geometry>
-                <cylinder radius="0.05" length="0.04"/>
+                <cylinder radius="0.035" length="0.028"/>
             </geometry>
             <material name="blue"/>
         </visual>
+        <collision>
+            <geometry>
+                <cylinder radius="0.035" length="0.028"/>
+            </geometry>
+        </collision>
+        <xacro:inertial_cylinder mass="0.1" length="0.028" radius="0.035">
+            <origin xyz="0.0 0.0 0.0" rpy="0.0 0.0 0.0"/>
+        </xacro:inertial_cylinder>
     </link>
-        <!-- RIGHT WHEEL LINK -->
+    <!-- RIGHT WHEEL LINK -->
+    <joint name="right_wheel_joint" type="continuous">
+        <origin xyz="0.0 -0.175 0.0" rpy="${pi/2} 0.0 0.0"/>
+        <parent link="base_link"/>
+        <child link="right_wheel"/>
+        <axis xyz="0.0 0.0 -1.0"/>
+        <limit lower="0.0" upper="0.0" effort="0.0" velocity="0.0"/>
+    </joint>
+    <link name="right_wheel">
+        <visual>
+            <geometry>
+                <cylinder radius="0.035" length="0.028"/>
+            </geometry>
+            <material name="blue"/>
+        </visual>
+        <collision>
+            <geometry>
+                <cylinder radius="0.035" length="0.028"/>
+            </geometry>
+        </collision>
+        <xacro:inertial_cylinder mass="0.1" length="0.028" radius="0.035">
+            <origin xyz="0.0 0.0 0.0" rpy="0.0 0.0 0.0"/>
+        </xacro:inertial_cylinder>
+    </link>
+    <!-- CASTER WHEEL FRONT LINK -->
+    <joint name="caster_wheel_front_joint" type="fixed">
+        <parent link="chassis"/>
+        <child link="caster_wheel_front"/>
+        <origin xyz="0.24 0.0 0.0"/>
+    </joint>
+    <link name="caster_wheel_front">
+        <visual>
+            <geometry>
+                <sphere radius="0.035"/>
+            </geometry>
+            <material name="black"/>
+        </visual>
+        <collision>
+            <geometry>
+                <sphere radius="0.035"/>
+            </geometry>
+        </collision>
+        <xacro:inertial_sphere mass="0.1" radius="0.035">
+            <origin xyz="0.0 0.0 0.0" rpy="0.0 0.0 0.0"/>
+        </xacro:inertial_sphere>
+    </link>
+    <!-- CASTER WHEEL REAR LINK -->
+    <joint name="caster_wheel_rear_joint" type="fixed">
+        <parent link="chassis"/>
+        <child link="caster_wheel_rear"/>
+        <origin xyz="0.05 0.0 0.0"/>
+    </joint>
+    <link name="caster_wheel_rear">
+        <visual>
+            <geometry>
+                <sphere radius="0.035"/>
+            </geometry>
+            <material name="black"/>
+        </visual>
+        <collision>
+            <geometry>
+                <sphere radius="0.035"/>
+            </geometry>
+        </collision>
+        <xacro:inertial_sphere mass="0.1" radius="0.035">
+            <origin xyz="0.0 0.0 0.0" rpy="0.0 0.0 0.0"/>
+        </xacro:inertial_sphere>
+    </link>
     <!-- Body Part
     <link name="body">

Commit message: created homebot urdf

File: description/robot_core.xacro (robot description, xacro)
@@ -18,4 +18,7 @@
         <color rgba="1 0.3 0.1 1"/>
     </material>
+    <material name="green">
+        <color rgba="0.0 1.0 0.0 1.0"/>
+    </material>
     <!-- BASE LINK -->
     <link name="base_link">
@@ -29,23 +32,23 @@
     <link name="chassis">
         <visual>
+            <origin xyz="0.15 0.0 0.02"/>
+            <geometry>
+                <cylinder radius="0.093" length="0.045"/>
+            </geometry>
+            <material name="orange"/>
+        </visual>
+        <collision>
             <origin xyz="0.15 0.0 0.075"/>
             <geometry>
-                <box size="0.3 0.3 0.15"/>
-            </geometry>
-            <material name="orange"/>
-        </visual>
-        <collision>
-            <origin xyz="0.15 0.0 0.075"/>
-            <geometry>
-                <box size="0.3 0.3 0.15"/>
-            </geometry>
-        </collision>
-        <xacro:inertial_box mass="0.5" x="0.3" y="0.3" z="0.15">
-            <origion xyz="0.15 0.0 0.075" rpy="0.0 0.0 0.0"/>
-        </xacro:inertial_box>
+                <cylinder radius="0.093" length="0.045"/>
+            </geometry>
+        </collision>
+        <xacro:inertial_cylinder mass="0.5" length="0.045" radius="0.093">
+            <origin xyz="0.0 0.0 0.0" rpy="0.0 0.0 0.0"/>
+        </xacro:inertial_cylinder>
     </link>
         <!-- LEFT WHEEL LINK -->
     <joint name="left_wheel_joint" type="continuous">
-        <origin xyz="0.0 0.175 0.0" rpy="-${pi/2} 0.0 0.0"/>
+        <origin xyz="0.0 0.11 0.0" rpy="-${pi/2} 0.0 0.0"/>
         <parent link="base_link"/>
         <child link="left_wheel"/>
@@ -71,5 +74,5 @@
     <!-- RIGHT WHEEL LINK -->
     <joint name="right_wheel_joint" type="continuous">
-        <origin xyz="0.0 -0.175 0.0" rpy="${pi/2} 0.0 0.0"/>
+        <origin xyz="0.0 -0.11 0.0" rpy="${pi/2} 0.0 0.0"/>
         <parent link="base_link"/>
         <child link="right_wheel"/>
@@ -95,21 +98,21 @@
     <!-- CASTER WHEEL FRONT LINK -->
     <joint name="caster_wheel_front_joint" type="fixed">
-        <parent link="chassis"/>
+        <parent link="base_link"/>
         <child link="caster_wheel_front"/>
-        <origin xyz="0.24 0.0 0.0"/>
+        <origin xyz="0.06 0.0 -0.015"/>
     </joint>
     <link name="caster_wheel_front">
         <visual>
             <geometry>
-                <sphere radius="0.035"/>
-            </geometry>
-            <material name="black"/>
-        </visual>
-        <collision>
-            <geometry>
-                <sphere radius="0.035"/>
-            </geometry>
-        </collision>
-        <xacro:inertial_sphere mass="0.1" radius="0.035">
+                <sphere radius="0.0155"/>
+            </geometry>
+            <material name="black"/>
+        </visual>
+        <collision>
+            <geometry>
+                <sphere radius="0.0155"/>
+            </geometry>
+        </collision>
+        <xacro:inertial_sphere mass="0.1" radius="0.0155">
             <origin xyz="0.0 0.0 0.0" rpy="0.0 0.0 0.0"/>
         </xacro:inertial_sphere>
@@ -117,25 +120,25 @@
     <!-- CASTER WHEEL REAR LINK -->
     <joint name="caster_wheel_rear_joint" type="fixed">
-        <parent link="chassis"/>
+        <parent link="base_link"/>
         <child link="caster_wheel_rear"/>
-        <origin xyz="0.05 0.0 0.0"/>
+        <origin xyz="-0.06 0.0 -0.015"/>
     </joint>
     <link name="caster_wheel_rear">
         <visual>
             <geometry>
-                <sphere radius="0.035"/>
-            </geometry>
-            <material name="black"/>
-        </visual>
-        <collision>
-            <geometry>
-                <sphere radius="0.035"/>
-            </geometry>
-        </collision>
-        <xacro:inertial_sphere mass="0.1" radius="0.035">
+                <sphere radius="0.0155"/>
+            </geometry>
+            <material name="black"/>
+        </visual>
+        <collision>
+            <geometry>
+                <sphere radius="0.0155"/>
+            </geometry>
+        </collision>
+        <xacro:inertial_sphere mass="0.1" radius="0.0155">
             <origin xyz="0.0 0.0 0.0" rpy="0.0 0.0 0.0"/>
         </xacro:inertial_sphere>
     </link>
-    <!-- Body Part
+    <!-- Body Part -->
     <link name="body">
         <visual>
@@ -143,13 +146,125 @@
                 <cylinder radius="0.11" length="0.345"/>
             </geometry>
-            <material name="yellow">
-            </material>
-        </visual>
+            <material name="yellow"/>
+        </visual>
+        <collision>
+            <geometry>
+                <cylinder radius="0.11" length="0.345"/>
+            </geometry>
+        </collision>
+        <xacro:inertial_cylinder mass="0.1" length="0.345" radius="0.11">
+            <origin xyz="0.0 0.0 0.0" rpy="0.0 0.0 0.0"/>
+        </xacro:inertial_cylinder>
     </link>
     <joint name="body_joint" type="fixed">
-        <parent link="chassis"/>
+        <parent link="base_link"/>
         <child link="body"/>
-        <origin xyz="0.0 0.0 0.17"/>
-    </joint>
--->
+        <origin xyz="0.0 0.0 0.21"/>
+    </joint>
+    <!-- LIDAR -->
+    <link name="lidar">
+        <visual>
+            <geometry>
+                <cylinder radius="0.035" length="0.02"/>
+            </geometry>
+            <material name="black"/>
+        </visual>
+        <collision>
+            <geometry>
+                <cylinder radius="0.035" length="0.02"/>
+            </geometry>
+            <material name="black"/>
+        </collision>
+        <xacro:inertial_cylinder mass="0.1" length="0.02" radius="0.035">
+            <origin xyz="0.0 0.0 0.0" rpy="0.0 0.0 0.0"/>
+        </xacro:inertial_cylinder>
+    </link>
+    <joint name="lidar_base_joint" type="fixed">
+        <parent link="base_link"/>
+        <child link="lidar"/>
+        <origin xyz="0.0 0.0 0.4"/>
+    </joint>
+    <!-- CAMERA -->
+    <link name="cam">
+        <visual>
+            <geometry>
+                <box size="0.03 0.03 0.03"/>
+            </geometry>
+            <material name="orange"/>
+        </visual>
+        <collision>
+            <geometry>
+                <box size="0.03 0.03 0.03"/>
+            </geometry>
+        </collision>
+        <xacro:inertial_box mass="0.1" x="0.03" y="0.03" z="0.03">
+            <origion xyz="0.0 0.0 0.0" rpy="0.0 0.0 0.0"/>
+        </xacro:inertial_box>
+    </link>
+    <joint name="cam_body_joint" type="fixed">
+        <origin xyz="0.1 0.0 0.06" rpy="${pi/2} 0.0 0.0"/>
+        <parent link="body"/>
+        <child link="cam"/>
+    </joint>
+    <link name="cam_linse">
+        <visual>
+            <geometry>
+                <cylinder radius="0.01" length="0.05"/>
+            </geometry>
+            <material name="black"/>
+        </visual>
+        <collision>
+            <geometry>
+                <cylinder radius="0.01" length="0.05"/>
+            </geometry>
+        </collision>
+    </link>
+    <joint name="linse_to_cam" type="fixed">
+        <origin xyz="0.0 0.0 0.0" rpy="0 ${pi/2} 0.0"/>
+        <parent link="cam"/>
+        <child link="cam_linse"/>
+    </joint>
+    <!-- LCD DISPLAY -->
+    <link name="display">
+        <visual>
+            <geometry>
+                <box size="0.09 0.09 0.05"/>
+            </geometry>
+            <material name="black"/>
+        </visual>
+        <collision>
+            <geometry>
+                <box size="0.09 0.09 0.03"/>
+            </geometry>
+        </collision>
+        <xacro:inertial_box mass="0.1" x="0.09" y="0.09" z="0.05">
+            <origion xyz="0.0 0.0 0.0" rpy="0.0 0.0 0.0"/>
+        </xacro:inertial_box>
+    </link>
+    <joint name="display_body_joint" type="fixed">
+        <origin xyz="0.08 0.0 0.11" rpy="0 0.0 0.0"/>
+        <parent link="body"/>
+        <child link="display"/>
+    </joint>
+    <link name="in_display">
+        <visual>
+            <geometry>
+                <box size="0.09 0.07 0.03"/>
+            </geometry>
+            <material name="green"/>
+        </visual>
+        <collision>
+            <geometry>
+                <box size="0.09 0.07 0.03"/>
+            </geometry>
+        </collision>
+        <xacro:inertial_box mass="0.1" x="0.09" y="0.09" z="0.03">
+            <origion xyz="0.0 0.0 0.0" rpy="0.0 0.0 0.0"/>
+        </xacro:inertial_box>
+    </link>
+    <joint name="in_display_body_joint" type="fixed">
+        <origin xyz="0.085 0.0 0.11" rpy="0 0.0 0.0"/>
+        <parent link="body"/>
+        <child link="in_display"/>
+    </joint>
 </robot>

Commit message: fixed base to chassis piont

File: description/robot_core.xacro (robot description, xacro)
@@ -28,9 +28,9 @@
         <parent link="base_link"/>
         <child link="chassis"/>
-        <origin xyz="-0.15 0.0 0.0"/>
+        <origin xyz="-0.093 0.0 0.0"/>
     </joint>
     <link name="chassis">
         <visual>
-            <origin xyz="0.15 0.0 0.02"/>
+            <origin xyz="0.093 0.0 0.02"/>
             <geometry>
                 <cylinder radius="0.093" length="0.045"/>
@@ -39,5 +39,5 @@
         </visual>
         <collision>
-            <origin xyz="0.15 0.0 0.075"/>
+            <origin xyz="0.093 0.0 0.075"/>
             <geometry>
                 <cylinder radius="0.093" length="0.045"/>
