Commit message: insert cam in gazebo

File: description/lidar.xacro (robot description, xacro)
@@ -31,5 +31,5 @@
             <sensor name="laser" type="ray">
                 <pose> 0 0 0 0 0 0 </pose>
-                <visualize>true</visualize>
+                <visualize>false</visualize>
                 <update_rate>10</update_rate>
                 <ray>

File: description/robot.urdf.xacro (robot description, xacro)
@@ -4,3 +4,4 @@
     <xacro:include filename="gazebo_control.xacro"/>
     <xacro:include filename="lidar.xacro"/>
+    <xacro:include filename="camera.xacro"/>
 </robot>

File: description/robot_core.xacro (robot description, xacro)
@@ -184,50 +184,4 @@
         <origin xyz="0.0 0.0 0.21"/>
     </joint>
-    <!-- CAMERA and Cam Linse-->
-    <link name="cam">
-        <visual>
-            <geometry>
-                <box size="0.03 0.03 0.03"/>
-            </geometry>
-            <material name="orange"/>
-        </visual>
-        <collision>
-            <geometry>
-                <box size="0.03 0.03 0.03"/>
-            </geometry>
-        </collision>
-        <xacro:inertial_box mass="0.1" x="0.03" y="0.03" z="0.03">
-            <origion xyz="0.0 0.0 0.0" rpy="0.0 0.0 0.0"/>
-        </xacro:inertial_box>
-    </link>
-    <gazebo reference="cam">
-        <material>Gazebo/Orange</material>
-    </gazebo>
-    <joint name="cam_body_joint" type="fixed">
-        <origin xyz="0.1 0.0 0.06" rpy="${pi/2} 0.0 0.0"/>
-        <parent link="body"/>
-        <child link="cam"/>
-    </joint>
-    <link name="cam_linse">
-        <visual>
-            <geometry>
-                <cylinder radius="0.01" length="0.05"/>
-            </geometry>
-            <material name="black"/>
-        </visual>
-        <collision>
-            <geometry>
-                <cylinder radius="0.01" length="0.05"/>
-            </geometry>
-        </collision>
-    </link>
-    <gazebo reference="cam_linse">
-        <material>Gazebo/Black</material>
-    </gazebo>
-    <joint name="linse_to_cam" type="fixed">
-        <origin xyz="0.0 0.0 0.0" rpy="0 ${pi/2} 0.0"/>
-        <parent link="cam"/>
-        <child link="cam_linse"/>
-    </joint>
     <!-- LCD DISPLAY and In_display  -->
     <link name="display">

Commit message: workflow

File: description/lidar.xacro (robot description, xacro)
@@ -25,5 +25,5 @@
             <parent link="base_link"/>
             <child link="laser_frame"/>
-            <origin xyz="0.0 0.0 0.4"/>
+            <origin xyz="0.0 0.0 0.4" rpy="0.0 0.0 -1.57"/>
         </joint>
         <gazebo reference="laser_frame">
@@ -31,5 +31,5 @@
             <sensor name="laser" type="ray">
                 <pose> 0 0 0 0 0 0 </pose>
-                <visualize>false</visualize>
+                <visualize>true</visualize>
                 <update_rate>10</update_rate>
                 <ray>
@@ -37,5 +37,6 @@
                         <horizontal>
                             <samples>360</samples>
-                            <min_angle>-3.14</min_angle>
+                            <resolution>1</resolution>
+                            <min_angle>0.00</min_angle>
                             <max_angle>3.14</max_angle>
                         </horizontal>
@@ -43,10 +44,10 @@
                     <range>
                         <min>0.3</min>
-                        <max>12</max>
+                        <max>6</max>
                     </range>
                 </ray>
                 <plugin name="laser_controller" filename="libgazebo_ros_ray_sensor.so">
                     <ros>
-                        <argument>--ros-args --remap ~/out:=scan</argument>
+                        <argument>~/out:=scan</argument>
                     </ros>
                     <output_type>sensor_msgs/LaserScan</output_type>

File: description/ros2_control.xacro (robot description, xacro)
@@ -15,6 +15,6 @@
             <joint name="left_wheel_joint">
                 <command_interface name="velocity">
-                    <param name="min">-30</param>
-                    <param name="max">30</param>
+                    <param name="min">-10</param>
+                    <param name="max">10</param>
                 </command_interface>
                 <state_interface name="velocity"/>
@@ -23,6 +23,6 @@
             <joint name="right_wheel_joint">
                 <command_interface name="velocity">
-                    <param name="min">-30</param>
-                    <param name="max">30</param>
+                    <param name="min">-10</param>
+                    <param name="max">10</param>
                 </command_interface>
                 <state_interface name="velocity"/>
