Commit message: save this

File: description/camera.xacro (robot description, xacro)
@@ -1,31 +1,53 @@
 <?xml version="1.0"?>
-<robot xmlns:xacro="http://www.ros.org/wiki/xacro">
-    <!-- Cam-->
-    <joint name="cam_joint" type="fixed">
-        <parent link="chassis"/>
-        <child link="cam"/>
-        <origin xyz="-0.04 0 0.138 "/>
-    </joint>
+<robot xmlns:xacro="http://www.ros.org/wiki/xacro" >
+<!-- CAMERA and Cam Linse-->
     <link name="cam">
         <visual>
-            <origin xyz="0.0 0.0 0.0" rpy="0.0 0.0 0.0"/>
             <geometry>
-                <box size="0.04 0.11 0.07"/>
+                <box size="0.03 0.03 0.03"/>
             </geometry>
-            <material name="white"/>
+            <material name="orange"/>
         </visual>
         <collision>
-            <origin xyz="0.0 0.0 0.0" rpy="0.0 0.0 0.0"/>
             <geometry>
-                <box size="0.04 0.11 0.07"/>
+                <box size="0.03 0.03 0.03"/>
             </geometry>
         </collision>
-        <xacro:inertial_box mass="0.2" x="0.04" y="0.11" z="0.07">
-            <origin xyz="0.0 0.0 0.0" rpy="0.0 0.0 0.0"/>
+        <xacro:inertial_box mass="0.1" x="0.03" y="0.03" z="0.03">
+            <origion xyz="0.0 0.0 0.0" rpy="0.0 0.0 0.0"/>
         </xacro:inertial_box>
     </link>
-    <gazebo reference="cam">
-        <material>Gazebo/White</material>
+    <link name="cam_linse">
+        <visual>
+            <geometry>
+                <cylinder radius="0.01" length="0.05"/>
+            </geometry>
+            <material name="black"/>
+        </visual>
+        <collision>
+            <geometry>
+                <cylinder radius="0.01" length="0.05"/>
+            </geometry>
+        </collision>
+    </link>
+    <link name="camera_link_optical"></link>
+    <gazebo reference="cam_linse">
+        <material>Gazebo/Black</material>
     </gazebo>
+    <joint name="cam_body_joint" type="fixed">
+        <origin xyz="0.1 0.0 0.06" rpy="${pi/2} 0.0 0.0"/>
+        <parent link="body"/>
+        <child link="cam"/>
+    </joint>
+    <joint name="linse_to_cam" type="fixed">
+        <origin xyz="0.0 0.0 0.0" rpy="0 ${pi/2} 0.0"/>
+        <parent link="cam"/>
+        <child link="cam_linse"/>
+    </joint>
+    <joint name="camera_optical_joint" type="fixed">
+        <origin xyz="0 0.0 0.0" rpy="${-pi/2} 0.0 ${-pi/2}"/>
+        <parent link="cam"/>
+        <child link="camera_link_optical"/>
+    </joint>
     <gazebo reference="cam">
         <material>Gazebo/Orange</material>
@@ -43,5 +65,5 @@
                 <clip>
                     <near>0.05</near>
-                    <far>7.0</far>
+                    <far>8.0</far>
                 </clip>
             </camera>

File: description/lidar.xacro (robot description, xacro)
@@ -1,4 +1,4 @@
 <?xml version="1.0"?>
-<robot xmlns:xacro="http://www.ros.org/wiki/xacro">
+<robot xmlns:xacro="http://www.ros.org/wiki/xacro" >
         <!-- LIDAR -->
         <link name="laser_frame">
@@ -25,25 +25,11 @@
             <parent link="base_link"/>
             <child link="laser_frame"/>
-            <origin xyz="0.0 0.0 0.4"/>
+            <origin xyz="0.0 0.0 0.4" rpy="0.0 0.0 -1.57"/>
         </joint>
-    <link name="lidar">
-        <visual>
-            <geometry>
-                <cylinder radius="0.06" length="0.04"/>
-            </geometry>
-            <material name="red"/>
-        </visual>
-        <collision>
-            <geometry>
-                <cylinder radius="0.06" length="0.04"/>
-            </geometry>
-        </collision>
-        <xacro:inertial_cylinder mass="0.01" radius="0.06" length="0.04">
-            <origin xyz="0.0 0.0 0.0" rpy="0.0 0.0 0.0"/>
-        </xacro:inertial_cylinder>
-    </link>
+        <gazebo reference="laser_frame">
+            <material>Gazebo/Black</material>
             <sensor name="laser" type="ray">
                 <pose> 0 0 0 0 0 0 </pose>
-                <visualize>false</visualize>
+                <visualize>true</visualize>
                 <update_rate>10</update_rate>
                 <ray>
@@ -51,5 +37,6 @@
                         <horizontal>
                             <samples>360</samples>
-                            <min_angle>-3.14</min_angle>
+                            <resolution>1</resolution>
+                            <min_angle>0.00</min_angle>
                             <max_angle>3.14</max_angle>
                         </horizontal>
@@ -57,10 +44,10 @@
                     <range>
                         <min>0.3</min>
-                        <max>12</max>
+                        <max>6</max>
                     </range>
                 </ray>
                 <plugin name="laser_controller" filename="libgazebo_ros_ray_sensor.so">
                     <ros>
-                        <argument>--ros-args --remap ~/out:=scan</argument>
+                        <argument>~/out:=scan</argument>
                     </ros>
                     <output_type>sensor_msgs/LaserScan</output_type>

File: description/robot_core.xacro (robot description, xacro)
@@ -28,11 +28,11 @@
         <parent link="base_link"/>
         <child link="chassis"/>
-        <origin xyz="-0.017 0.0 0.0"/>
+        <origin xyz="-0.093 0.0 0.0"/>
     </joint>
     <link name="chassis">
         <visual>
-            <origin xyz="0.017 0.0 0.017"/>
-            <geometry>
-                <box size="0.034 0.25 0.034"/>
+            <origin xyz="0.093 0.0 0.02"/>
+            <geometry>
+                <cylinder radius="0.093" length="0.045"/>
             </geometry>
             <material name="orange"/>
@@ -41,17 +41,17 @@
             <origin xyz="0.093 0.0 0.075"/>
             <geometry>
-                <box size="0.034 0.25 0.034"/>
-            </geometry>
-        </collision>
-        <xacro:inertial_box mass="1.5" x="0.034" y="0.25" z="0.034">
-            <origin xyz="0.0 0.0 0.0" rpy="0.0 0.0 0.0"/>
-        </xacro:inertial_box>
+                <cylinder radius="0.093" length="0.045"/>
+            </geometry>
+        </collision>
+        <xacro:inertial_cylinder mass="0.5" length="0.045" radius="0.093">
+            <origin xyz="0.0 0.0 0.0" rpy="0.0 0.0 0.0"/>
+        </xacro:inertial_cylinder>
     </link>
     <gazebo reference="chassis">
-        <material>Gazebo/Black</material>
+        <material>Gazebo/Orange</material>
     </gazebo>
         <!-- LEFT WHEEL LINK -->
     <joint name="left_wheel_joint" type="continuous">
-        <origin xyz="0 -0.128 0.017" rpy="${pi/2} 0 0"/>
+        <origin xyz="0.0 0.11 0.0" rpy="-${pi/2} 0.0 0.0"/>
         <parent link="base_link"/>
         <child link="left_wheel"/>
@@ -62,5 +62,5 @@
         <visual>
             <geometry>
-                <cylinder radius="0.06" length="0.04"/>
+                <cylinder radius="0.035" length="0.028"/>
             </geometry>
             <material name="blue"/>
@@ -68,8 +68,8 @@
         <collision>
             <geometry>
-                <cylinder radius="0.06" length="0.04"/>
-            </geometry>
-        </collision>
-        <xacro:inertial_cylinder mass="0.1" length="0.04" radius="0.06">
+                <cylinder radius="0.035" length="0.028"/>
+            </geometry>
+        </collision>
+        <xacro:inertial_cylinder mass="0.1" length="0.028" radius="0.035">
             <origin xyz="0.0 0.0 0.0" rpy="0.0 0.0 0.0"/>
         </xacro:inertial_cylinder>
@@ -78,7 +78,7 @@
         <material>Gazebo/Blue</material>
     </gazebo>
-    <!-- RIGHT WHEEL  LINK -->
+    <!-- RIGHT WHEEL LINK -->
     <joint name="right_wheel_joint" type="continuous">
-        <origin xyz="0 0.128 0.017" rpy="-${pi/2} 0 0"/>
+        <origin xyz="0.0 -0.11 0.0" rpy="${pi/2} 0.0 0.0"/>
         <parent link="base_link"/>
         <child link="right_wheel"/>
@@ -89,5 +89,5 @@
         <visual>
             <geometry>
-                <cylinder radius="0.06" length="0.04"/>
+                <cylinder radius="0.035" length="0.028"/>
             </geometry>
             <material name="blue"/>
@@ -95,8 +95,8 @@
         <collision>
             <geometry>
-                <cylinder radius="0.06" length="0.04"/>
-            </geometry>
-        </collision>
-        <xacro:inertial_cylinder mass="0.1" length="0.04" radius="0.06">
+                <cylinder radius="0.035" length="0.028"/>
+            </geometry>
+        </collision>
+        <xacro:inertial_cylinder mass="0.1" length="0.028" radius="0.035">
             <origin xyz="0.0 0.0 0.0" rpy="0.0 0.0 0.0"/>
         </xacro:inertial_cylinder>
@@ -105,112 +105,131 @@
         <material>Gazebo/Blue</material>
     </gazebo>
-    <!-- Caster Wheel Holder and Caster Wheel -->
-    <joint name="caster_wheel_holder_joint" type="fixed">
-        <parent link="chassis"/>
-        <child link="caster_wheel_holder"/>
-        <origin xyz="0.25 0.0 0.0"/>
-    </joint>
-    <link name="caster_wheel_holder">
-        <visual>
-            <origin xyz="0.0 0.0 0.017"/>
-            <geometry>
-                <box size="0.034 0.034 0.034"/>
+    <!-- CASTER WHEEL FRONT LINK -->
+    <joint name="caster_wheel_front_joint" type="fixed">
+        <parent link="base_link"/>
+        <child link="caster_wheel_front"/>
+        <origin xyz="0.085 0.0 -0.016"/>
+    </joint>
+    <link name="caster_wheel_front">
+        <visual>
+            <geometry>
+                <sphere radius="0.018"/>
             </geometry>
             <material name="black"/>
         </visual>
         <collision>
-            <origin xyz="0.0 0.0 0.017"/>
-            <geometry>
-                <box size="0.034 0.034 0.034"/>
-            </geometry>
-        </collision>
-        <xacro:inertial_box mass="1.5" x="0.034" y="0.034" z="0.034">
-            <origin xyz="0.0 0.0 0.0" rpy="0.0 0.0 0.0"/>
-        </xacro:inertial_box>
-    </link>
-    <gazebo reference="caster_wheel_holder">
+            <geometry>
+                <sphere radius="0.018"/>
+            </geometry>
+        </collision>
+        <xacro:inertial_sphere mass="0.3" radius="0.018">
+            <origin xyz="0.0 0.0 0.0" rpy="0.0 0.0 0.0"/>
+        </xacro:inertial_sphere>
+    </link>
+    <gazebo reference="caster_wheel_front">
         <material>Gazebo/Black</material>
-    </gazebo>
-    <!-- caster Wheel-->
-    <joint name="caster_wheel_joint" type="fixed">
-        <parent link="caster_wheel_holder"/>
-        <child link="caster_wheel_link"/>
-        <origin xyz="0.0 0.0 -0.017"/>
-    </joint>
-    <link name="caster_wheel_link">
-        <visual>
-            <geometry>
-                <sphere radius="0.03"/>
-            </geometry>
-            <material name="blue">
-            </material>
-        </visual>
-        <collision>
-            <geometry>
-                <sphere radius="0.03"/>
-            </geometry>
-        </collision>
-        <xacro:inertial_sphere mass="0.15" radius="0.03">
-            <origin xyz="0.0 0.0 0.0" rpy="0.0 0.0 0.0"/>
-        </xacro:inertial_sphere>
-    </link>
-    <gazebo reference="caster_wheel_link">
-        <material>Gazebo/Blue</material>
         <mu1 value="0.001"/>
         <mu2 value="0.001"/>
     </gazebo>
-    <!-- BODY PARTS-->
+    <!-- CASTER WHEEL REAR LINK -->
+    <joint name="caster_wheel_rear_joint" type="fixed">
+        <parent link="base_link"/>
+        <child link="caster_wheel_rear"/>
+        <origin xyz="-0.085 0.0 -0.0165"/>
+    </joint>
+    <link name="caster_wheel_rear">
+        <visual>
+            <geometry>
+                <sphere radius="0.018"/>
+            </geometry>
+            <material name="black"/>
+        </visual>
+        <collision>
+            <geometry>
+                <sphere radius="0.018"/>
+            </geometry>
+        </collision>
+        <xacro:inertial_sphere mass="0.3" radius="0.018">
+            <origin xyz="0.0 0.0 0.0" rpy="0.0 0.0 0.0"/>
+        </xacro:inertial_sphere>
+    </link>
+    <gazebo reference="caster_wheel_rear">
+        <material>Gazebo/Black</material>
+        <mu1 value="0.001"/>
+        <mu2 value="0.001"/>
+    </gazebo>
+    <!-- Body Part -->
+    <link name="body">
+        <visual>
+            <geometry>
+                <cylinder radius="0.11" length="0.345"/>
+            </geometry>
+            <material name="yellow"/>
+        </visual>
+        <collision>
+            <geometry>
+                <cylinder radius="0.11" length="0.345"/>
+            </geometry>
+        </collision>
+        <xacro:inertial_cylinder mass="0.1" length="0.345" radius="0.11">
+            <origin xyz="0.0 0.0 0.0" rpy="0.0 0.0 0.0"/>
+        </xacro:inertial_cylinder>
+    </link>
+    <gazebo reference="body">
+        <material>Gazebo/Yellow</material>
+    </gazebo>
     <joint name="body_joint" type="fixed">
-        <parent link="chassis"/>
+        <parent link="base_link"/>
         <child link="body"/>
-        <origin xyz="0.110 0.0 0.069"/>
-    </joint>
-    <link name="body">
-        <visual>
-            <origin xyz="0.0 0.0 0.0"/>
-            <geometry>
-                <box size="0.4 0.11 0.07"/>
-            </geometry>
-            <material name="orange"/>
-        </visual>
-        <collision>
-            <origin xyz="0.093 0.0 0.075"/>
-            <geometry>
-                <box size="0.4 0.11 0.07"/>
-            </geometry>
-        </collision>
-        <xacro:inertial_box mass="0.5" x="0.4" y="0.11" z="0.07">
-            <origin xyz="0.0 0.0 0.0" rpy="0.0 0.0 0.0"/>
+        <origin xyz="0.0 0.0 0.21"/>
+    </joint>
+    <!-- LCD DISPLAY and In_display  -->
+    <link name="display">
+        <visual>
+            <geometry>
+                <box size="0.09 0.09 0.05"/>
+            </geometry>
+            <material name="black"/>
+        </visual>
+        <collision>
+            <geometry>
+                <box size="0.09 0.09 0.03"/>
+            </geometry>
+        </collision>
+        <xacro:inertial_box mass="0.1" x="0.09" y="0.09" z="0.05">
+            <origion xyz="0.0 0.0 0.0" rpy="0.0 0.0 0.0"/>
         </xacro:inertial_box>
     </link>
-    <gazebo reference="body">
-        <material>Gazebo/Orange</material>
-    </gazebo>
-    <!-- BodyTop-->
-    <joint name="body_top_joint" type="fixed">
-        <parent link="chassis"/>
-        <child link="body_top"/>
-        <origin xyz="0.16 0.0 0.138"/>
-    </joint>
-    <link name="body_top">
-        <visual>
-            <origin xyz="0.0 0.0 0.0"/>
-            <geometry>
-                <box size="0.3 0.11 0.07"/>
-            </geometry>
-            <material name="orange"/>
-        </visual>
-        <collision>
-            <origin xyz="0.093 0.0 0.075"/>
-            <geometry>
-                <box size="0.4 0.11 0.07"/>
-            </geometry>
-        </collision>
-        <xacro:inertial_box mass="0.5" x="0.4" y="0.11" z="0.07">
-            <origin xyz="0.0 0.0 0.0" rpy="0.0 0.0 0.0"/>
+    <gazebo reference="display">
+        <material>Gazebo/Black</material>
+    </gazebo>
+    <joint name="display_body_joint" type="fixed">
+        <origin xyz="0.08 0.0 0.11" rpy="0 0.0 0.0"/>
+        <parent link="body"/>
+        <child link="display"/>
+    </joint>
+    <link name="in_display">
+        <visual>
+            <geometry>
+                <box size="0.09 0.07 0.03"/>
+            </geometry>
+            <material name="green"/>
+        </visual>
+        <collision>
+            <geometry>
+                <box size="0.09 0.07 0.03"/>
+            </geometry>
+        </collision>
+        <xacro:inertial_box mass="0.1" x="0.09" y="0.09" z="0.03">
+            <origion xyz="0.0 0.0 0.0" rpy="0.0 0.0 0.0"/>
         </xacro:inertial_box>
     </link>
-    <gazebo reference="body_top">
-        <material>Gazebo/Orange</material>
-    </gazebo>
+    <gazebo reference="in_display">
+        <material>Gazebo/Green</material>
+    </gazebo>
+    <joint name="in_display_body_joint" type="fixed">
+        <origin xyz="0.085 0.0 0.11" rpy="0 0.0 0.0"/>
+        <parent link="body"/>
+        <child link="in_display"/>
+    </joint>
 </robot>

File: description/ros2_control.xacro (robot description, xacro)
@@ -11,5 +11,5 @@
                 <param name="baud_rate">57600</param>
                 <param name="timeout">1000</param>
-                <param name="enc_counts_per_rev">408</param>
+                <param name="enc_counts_per_rev">426</param>
             </hardware>
             <joint name="left_wheel_joint">
@@ -56,6 +56,6 @@
     <gazebo>
         <plugin name="gazebo_ros2_control" filename="libgazebo_ros2_control.so">
-            <parameters>$(find scout)/config/my_controllers.yaml</parameters>
-            <parameters>$(find scout)/config/gaz_ros2_ctl_use_sim.yaml</parameters>
+            <parameters>$(find homerobot)/config/my_controllers.yaml</parameters>
+            <parameters>$(find homerobot)/config/gaz_ros2_ctl_use_sim.yaml</parameters>
         </plugin>
     </gazebo>
