Commit message: working on xacro urdf

File: description/robot.urdf.xacro (robot description, xacro)
@@ -1,5 +1,4 @@
 <?xml version="1.0"?>
 <robot xmlns:xacro="http://www.ros.org/wiki/xacro"  name="homebot">
-    <!-- Example link -->
-    <link name="base_link"></link>
+    <xacro:include filename="robot_core.xacro"/>
 </robot>

Commit message: workflow gazebo and lidar in gazebo

File: description/robot.urdf.xacro (robot description, xacro)
@@ -2,3 +2,5 @@
 <robot xmlns:xacro="http://www.ros.org/wiki/xacro"  name="homebot">
     <xacro:include filename="robot_core.xacro"/>
+    <xacro:include filename="gazebo_control.xacro"/>
+    <xacro:include filename="lidar.xacro"/>
 </robot>

File: description/robot_core.xacro (robot description, xacro)
@@ -48,4 +48,7 @@
         </xacro:inertial_cylinder>
     </link>
+    <gazebo reference="chassis">
+        <material>Gazebo/Orange</material>
+    </gazebo>
         <!-- LEFT WHEEL LINK -->
     <joint name="left_wheel_joint" type="continuous">
@@ -72,4 +75,7 @@
         </xacro:inertial_cylinder>
     </link>
+    <gazebo reference="left_wheel">
+        <material>Gazebo/Blue</material>
+    </gazebo>
     <!-- RIGHT WHEEL LINK -->
     <joint name="right_wheel_joint" type="continuous">
@@ -96,48 +102,61 @@
         </xacro:inertial_cylinder>
     </link>
+    <gazebo reference="right_wheel">
+        <material>Gazebo/Blue</material>
+    </gazebo>
     <!-- CASTER WHEEL FRONT LINK -->
     <joint name="caster_wheel_front_joint" type="fixed">
         <parent link="base_link"/>
         <child link="caster_wheel_front"/>
-        <origin xyz="0.06 0.0 -0.015"/>
+        <origin xyz="0.085 0.0 -0.016"/>
     </joint>
     <link name="caster_wheel_front">
         <visual>
             <geometry>
-                <sphere radius="0.0155"/>
-            </geometry>
-            <material name="black"/>
-        </visual>
-        <collision>
-            <geometry>
-                <sphere radius="0.0155"/>
-            </geometry>
-        </collision>
-        <xacro:inertial_sphere mass="0.1" radius="0.0155">
+                <sphere radius="0.018"/>
+            </geometry>
+            <material name="black"/>
+        </visual>
+        <collision>
+            <geometry>
+                <sphere radius="0.018"/>
+            </geometry>
+        </collision>
+        <xacro:inertial_sphere mass="0.3" radius="0.018">
             <origin xyz="0.0 0.0 0.0" rpy="0.0 0.0 0.0"/>
         </xacro:inertial_sphere>
     </link>
+    <gazebo reference="caster_wheel_front">
+        <material>Gazebo/Black</material>
+        <mu1 value="0.001"/>
+        <mu2 value="0.001"/>
+    </gazebo>
     <!-- CASTER WHEEL REAR LINK -->
     <joint name="caster_wheel_rear_joint" type="fixed">
         <parent link="base_link"/>
         <child link="caster_wheel_rear"/>
-        <origin xyz="-0.06 0.0 -0.015"/>
+        <origin xyz="-0.085 0.0 -0.0165"/>
     </joint>
     <link name="caster_wheel_rear">
         <visual>
             <geometry>
-                <sphere radius="0.0155"/>
-            </geometry>
-            <material name="black"/>
-        </visual>
-        <collision>
-            <geometry>
-                <sphere radius="0.0155"/>
-            </geometry>
-        </collision>
-        <xacro:inertial_sphere mass="0.1" radius="0.0155">
+                <sphere radius="0.018"/>
+            </geometry>
+            <material name="black"/>
+        </visual>
+        <collision>
+            <geometry>
+                <sphere radius="0.018"/>
+            </geometry>
+        </collision>
+        <xacro:inertial_sphere mass="0.3" radius="0.018">
             <origin xyz="0.0 0.0 0.0" rpy="0.0 0.0 0.0"/>
         </xacro:inertial_sphere>
     </link>
+    <gazebo reference="caster_wheel_rear">
+        <material>Gazebo/Black</material>
+        <mu1 value="0.001"/>
+        <mu2 value="0.001"/>
+    </gazebo>
     <!-- Body Part -->
     <link name="body">
@@ -157,4 +176,7 @@
         </xacro:inertial_cylinder>
     </link>
+    <gazebo reference="body">
+        <material>Gazebo/Yellow</material>
+    </gazebo>
     <joint name="body_joint" type="fixed">
         <parent link="base_link"/>
@@ -162,28 +184,5 @@
         <origin xyz="0.0 0.0 0.21"/>
     </joint>
-    <!-- LIDAR -->
-    <link name="lidar">
-        <visual>
-            <geometry>
-                <cylinder radius="0.035" length="0.02"/>
-            </geometry>
-            <material name="black"/>
-        </visual>
-        <collision>
-            <geometry>
-                <cylinder radius="0.035" length="0.02"/>
-            </geometry>
-            <material name="black"/>
-        </collision>
-        <xacro:inertial_cylinder mass="0.1" length="0.02" radius="0.035">
-            <origin xyz="0.0 0.0 0.0" rpy="0.0 0.0 0.0"/>
-        </xacro:inertial_cylinder>
-    </link>
-    <joint name="lidar_base_joint" type="fixed">
-        <parent link="base_link"/>
-        <child link="lidar"/>
-        <origin xyz="0.0 0.0 0.4"/>
-    </joint>
-    <!-- CAMERA -->
+    <!-- CAMERA and Cam Linse-->
     <link name="cam">
         <visual>
@@ -202,4 +201,7 @@
         </xacro:inertial_box>
     </link>
+    <gazebo reference="cam">
+        <material>Gazebo/Orange</material>
+    </gazebo>
     <joint name="cam_body_joint" type="fixed">
         <origin xyz="0.1 0.0 0.06" rpy="${pi/2} 0.0 0.0"/>
@@ -220,4 +222,7 @@
         </collision>
     </link>
+    <gazebo reference="cam_linse">
+        <material>Gazebo/Black</material>
+    </gazebo>
     <joint name="linse_to_cam" type="fixed">
         <origin xyz="0.0 0.0 0.0" rpy="0 ${pi/2} 0.0"/>
@@ -225,5 +230,5 @@
         <child link="cam_linse"/>
     </joint>
-    <!-- LCD DISPLAY -->
+    <!-- LCD DISPLAY and In_display  -->
     <link name="display">
         <visual>
@@ -242,4 +247,7 @@
         </xacro:inertial_box>
     </link>
+    <gazebo reference="display">
+        <material>Gazebo/Black</material>
+    </gazebo>
     <joint name="display_body_joint" type="fixed">
         <origin xyz="0.08 0.0 0.11" rpy="0 0.0 0.0"/>
@@ -263,4 +271,7 @@
         </xacro:inertial_box>
     </link>
+    <gazebo reference="in_display">
+        <material>Gazebo/Green</material>
+    </gazebo>
     <joint name="in_display_body_joint" type="fixed">
         <origin xyz="0.085 0.0 0.11" rpy="0 0.0 0.0"/>

Commit message: working on real robot

File: description/robot.urdf.xacro (robot description, xacro)
@@ -2,4 +2,5 @@
 <robot xmlns:xacro="http://www.ros.org/wiki/xacro"  name="homebot">
     <xacro:arg name="use_ros2_control" default="true"/>
+    <xacro:arg name="sim_mode" default="false"/>
     <xacro:include filename="robot_core.xacro"/>
     <xacro:if value="$(arg use_ros2_control)">

File: description/ros2_control.xacro (robot description, xacro)
@@ -1,28 +1,61 @@
 <?xml version="1.0"?>
 <robot xmlns:xacro="http://www.ros.org/wiki/xacro">
-    <ros2_control name="GazeboSystem" type="system">
-        <hardware>
-            <plugin>gazebo_ros2_control/GazeboSystem</plugin>
-        </hardware>
-        <joint name="left_wheel_joint">
-            <command_interface name="velocity">
-                <param name="min">-10</param>
-                <param name="max">10</param>
-            </command_interface>
-            <state_interface name="velocity"/>
-            <state_interface name="position"/>
-        </joint>
-        <joint name="right_wheel_joint">
-            <command_interface name="velocity">
-                <param name="min">-10</param>
-                <param name="max">10</param>
-            </command_interface>
-            <state_interface name="velocity"/>
-            <state_interface name="position"/>
-        </joint>
-    </ros2_control>
+    <xacro:unless value="$(arg sim_mode)">
+        <ros2_control name="RealRobot" type="system">
+            <hardware>
+                <plugin>diffdrive_arduino/DiffDriveArduino</plugin>
+                <param name="left_wheel_name">left_wheel_joint</param>
+                <param name="right_wheel_name">right_wheel_joint</param>
+                <param name="loop_rate">30</param>
+                <param name="device">/dev/ttyUSB0</param>
+                <param name="baud_rate">57600</param>
+                <param name="timeout">1000</param>
+                <param name="enc_counts_per_rev">426</param>
+            </hardware>
+            <joint name="left_wheel_joint">
+                <command_interface name="velocity">
+                    <param name="min">-10</param>
+                    <param name="max">10</param>
+                </command_interface>
+                <state_interface name="velocity"/>
+                <state_interface name="position"/>
+            </joint>
+            <joint name="right_wheel_joint">
+                <command_interface name="velocity">
+                    <param name="min">-10</param>
+                    <param name="max">10</param>
+                </command_interface>
+                <state_interface name="velocity"/>
+                <state_interface name="position"/>
+            </joint>
+        </ros2_control>
+    </xacro:unless>
+    <xacro:if value="$(arg sim_mode)">
+        <ros2_control name="GazeboSystem" type="system">
+            <hardware>
+                <plugin>gazebo_ros2_control/GazeboSystem</plugin>
+            </hardware>
+            <joint name="left_wheel_joint">
+                <command_interface name="velocity">
+                    <param name="min">-10</param>
+                    <param name="max">10</param>
+                </command_interface>
+                <state_interface name="velocity"/>
+                <state_interface name="position"/>
+            </joint>
+            <joint name="right_wheel_joint">
+                <command_interface name="velocity">
+                    <param name="min">-10</param>
+                    <param name="max">10</param>
+                </command_interface>
+                <state_interface name="velocity"/>
+                <state_interface name="position"/>
+            </joint>
+        </ros2_control>
+    </xacro:if>
     <gazebo>
         <plugin name="gazebo_ros2_control" filename="libgazebo_ros2_control.so">
             <parameters>$(find homerobot)/config/my_controllers.yaml</parameters>
+            <parameters>$(find homerobot)/config/gaz_ros2_ctl_use_sim.yaml</parameters>
         </plugin>
     </gazebo>

Commit message: missing odom

File: description/robot.urdf.xacro (robot description, xacro)
@@ -1,7 +1,13 @@
 <?xml version="1.0"?>
 <robot xmlns:xacro="http://www.ros.org/wiki/xacro"  name="homebot">
+<!--
     <xacro:arg name="use_ros2_control" default="false"/>
     <xacro:arg name="sim_mode" default="true"/>
+-->
     <xacro:include filename="robot_core.xacro"/>
+    <xacro:include filename="lidar.xacro"/>
+    <xacro:include filename="camera.xacro"/>
+    <xacro:include filename="gazebo_control.xacro"/>
+    <!--
     <xacro:if value="$(arg use_ros2_control)">
         <xacro:include filename="ros2_control.xacro"/>
@@ -10,5 +16,4 @@
         <xacro:include filename="gazebo_control.xacro"/>
     </xacro:unless>
-    <xacro:include filename="lidar.xacro"/>
-    <xacro:include filename="camera.xacro"/>
+    -->
 </robot>

File: description/robot_core.xacro (robot description, xacro)
@@ -24,4 +24,12 @@
     <link name="base_link">
     </link>
+    <!-- BASE FOOT PRINT -->
+    <joint name="base_footprint_joint" type="fixed">
+        <parent link="base_link"/>
+        <child link="base_footprint"/>
+        <origin xyz="0.0 0.0 0.0" rpy="0.0 0.0 0.0"/>
+    </joint>
+    <link name="base_footprint">
+    </link>
     <!-- CHASSIS LINK -->
     <joint name="cassis_joint" type="fixed">
@@ -53,5 +61,5 @@
         <!-- LEFT WHEEL LINK -->
     <joint name="left_wheel_joint" type="continuous">
-        <origin xyz="0.0 0.11 0.0" rpy="-${pi/2} 0.0 0.0"/>
+        <origin xyz="0.0 0.11 0.0" rpy="${-pi/2} 0.0 0.0"/>
         <parent link="base_link"/>
         <child link="left_wheel"/>
