Commit message: ...

File: description/gazebo_control.xacro (robot description, xacro)
@@ -3,4 +3,5 @@
     <gazebo>
         <plugin name="diff_drive" filename="libgazebo_ros_diff_drive.so">
+            <updateRate>30</updateRate>
             <!-- Reifen Infos -->
             <left_joint>left_wheel_joint</left_joint>

File: description/robot_core.xacro (robot description, xacro)
@@ -22,14 +22,12 @@
     </material>
     <!-- BASE LINK -->
-    <link name="base_link">
-    </link>
+    <link name="base_footprint"/>
+    <link name="base_link"/>
     <!-- BASE FOOT PRINT -->
     <joint name="base_footprint_joint" type="fixed">
-        <parent link="base_link"/>
-        <child link="base_footprint"/>
+        <parent link="base_footprint"/>
+        <child link="base_link"/>
         <origin xyz="0.0 0.0 0.0" rpy="0.0 0.0 0.0"/>
     </joint>
-    <link name="base_footprint">
-    </link>
     <!-- CHASSIS LINK -->
     <joint name="cassis_joint" type="fixed">

File: description/ros2_control.xacro (robot description, xacro)
@@ -18,6 +18,6 @@
                     <param name="max">10</param>
                 </command_interface>
-                <state_interface name="velocity"/>
-                <state_interface name="position"/>
+                <state_interface name="velocity" />
+                <state_interface name="position" />
             </joint>
             <joint name="right_wheel_joint">
@@ -26,6 +26,6 @@
                     <param name="max">10</param>
                 </command_interface>
-                <state_interface name="velocity"/>
-                <state_interface name="position"/>
+                <state_interface name="velocity" />
+                <state_interface name="position" />
             </joint>
         </ros2_control>
